Commit message: Stable

File: resources/robots/leg/leg.urdf (robot description, URDF)
Before this commit: robot leg7, 11 links, 10 joints
Links:
- link L_calf: geometry collision cylinder length=0.29 radius=0.040; visual mesh filename=meshes/L_calf.STL
- link L_thigh: geometry collision cylinder length=0.29 radius=0.040; visual mesh filename=meshes/L_thigh.STL
- link R_calf: geometry collision cylinder length=0.29 radius=0.040; visual mesh filename=meshes/R_calf.STL
- link R_thigh: geometry collision cylinder length=0.29 radius=0.040; visual mesh filename=meshes/R_thigh.STL
- link base: mass 8.0 -> 16.0
Joints:
- joint L_calf_joint: limit lower=0 upper=2 effort=500 velocity=50 -> lower=0 upper=2 effort=250 velocity=50
- joint L_hip2_joint: limit lower=-0.5 upper=1 effort=500 velocity=50 -> lower=-0.5 upper=1 effort=50 velocity=50
- joint L_hip_joint: limit lower=-1.5 upper=1.5 effort=500 velocity=50 -> lower=-1.5 upper=1.5 effort=50 velocity=50
- joint L_thigh_joint: limit lower=-1.7 upper=0 effort=500 velocity=50 -> lower=-1.7 upper=0 effort=100 velocity=50
- joint L_toe_joint: limit lower=-0.8 upper=0.8 effort=500 velocity=50 -> lower=-0.8 upper=0.8 effort=100 velocity=50
- joint R_calf_joint: limit lower=0 upper=2 effort=500 velocity=50 -> lower=0 upper=2 effort=250 velocity=50
- joint R_hip2_joint: limit lower=-1 upper=0.5 effort=500 velocity=50 -> lower=-1 upper=0.5 effort=50 velocity=50
- joint R_hip_joint: limit lower=-1.5 upper=1.5 effort=500 velocity=50 -> lower=-1.5 upper=1.5 effort=50 velocity=50
- joint R_thigh_joint: limit lower=-1.7 upper=0 effort=500 velocity=50 -> lower=-1.7 upper=0 effort=100 velocity=50
- joint R_toe_joint: limit lower=-0.8 upper=0.8 effort=500 velocity=50 -> lower=-0.8 upper=0.8 effort=100 velocity=50
